File: BeamBender-BigBox.kicad_pcb (KiCad board)
At the start: 4 copper layers, 157.5 x 90 mm, 163 parts, among them CN1 A4000-CN621-36, CN2 A4000-CN622-54, J1 HDMI, J2 JTAG, J3 JTAG_Pogo, J4 EXT_BUTTONS, J5 XAUDIO, J6 SJ1-3535NG, SW1 MENU, SW2 UP, SW3 DOWN, U1 Colorlight-i5-v7.0, U10 TPS2553DBVR, U2 TLV76133DCYR, U3 74LVC16244ADGG, U4 74LVC16244ADGG, U5 SII9022ACNU, U6 74LVC1G86, U7 AK5720VT, U8 AP2112K-1.2, U9 OPA1692, X1 Oscillator_3.2x2.5mm-27MHz, X2 Oscillator_5.0x3.2mm_24.576MHz

Commit message: Rev 0.3
Added test points for unused AV slot and FPGA pins
Added option to use Paula RAW audio
Parts:
- added R60: 0, Resistor_SMD:R_0603_1608Metric, B.Cu at (138.2, 65.1)
- added SJ1: LEFT, Jumper:SolderJumper-3_P1.3mm_Bridged12_RoundedPad1.0x1.5mm, B.Cu at (89.0, 60.0)
- added SJ2: RIGHT, Jumper:SolderJumper-3_P1.3mm_Bridged12_RoundedPad1.0x1.5mm, B.Cu at (99.2, 60.0)
- added TP1: TP_PPD7, TestPoint:TestPoint_Pad_D1.0mm, B.Cu at (195.6, 59.5)
- added TP10: TP_PBUSY, TestPoint:TestPoint_Pad_D1.0mm, B.Cu at (180.4, 59.5)
- added TP11: TP_PPOUT, TestPoint:TestPoint_Pad_D1.0mm, B.Cu at (177.8, 59.5)
- added TP12: TP_LED, TestPoint:TestPoint_Pad_D1.0mm, B.Cu at (197.3, 67.4)
- added TP13: TP_C3, TestPoint:TestPoint_Pad_D1.0mm, B.Cu at (179.5, 67.4)
- added TP14: TP_SOG, TestPoint:TestPoint_Pad_D1.0mm, B.Cu at (174.5, 67.4)
- added TP15: TP_TBASE, TestPoint:TestPoint_Pad_D1.0mm, B.Cu at (175.3, 59.5)
- added TP16: TP_C1, TestPoint:TestPoint_Pad_D1.0mm, B.Cu at (147.3, 60.4)
- added TP17: TP_XCLK, TestPoint:TestPoint_Pad_D1.0mm, B.Cu at (146.5, 67.4)
- added TP18: TP_BLANK, TestPoint:TestPoint_Pad_D1.0mm, B.Cu at (139.3, 60.4)
- added TP19: TP_C4, TestPoint:TestPoint_Pad_D1.0mm, B.Cu at (128.7, 67.4)
- added TP2: TP_PPD6, TestPoint:TestPoint_Pad_D1.0mm, B.Cu at (194.3, 67.4)
- added TP20: TP_XCLKEN, TestPoint:TestPoint_Pad_D1.0mm, B.Cu at (124.5, 60.4)
- added TP21: TP_ABLUE, TestPoint:TestPoint_Pad_D1.0mm, B.Cu at (123.7, 67.4)
- added TP22: TP_AGREEN, TestPoint:TestPoint_Pad_D1.0mm, B.Cu at (118.6, 67.4)
- added TP23: TP_ARED, TestPoint:TestPoint_Pad_D1.0mm, B.Cu at (113.5, 67.4)
- added TP24: TP_SPARE_IN5, TestPoint:TestPoint_Pad_D1.0mm, B.Cu at (139.0, 67.4)
- added TP25: TP_SPARE_OUT3, TestPoint:TestPoint_Pad_D1.0mm, B.Cu at (137.2, 74.5)
- added TP26: TP_FPGA41, TestPoint:TestPoint_Pad_D1.0mm, B.Cu at (183.7, 93.5)
- added TP27: TP_FPGA79, TestPoint:TestPoint_Pad_D1.0mm, B.Cu at (172.3, 93.5)
- added TP28: TP_FPGA87, TestPoint:TestPoint_Pad_D1.0mm, B.Cu at (169.9, 93.5)
- added TP29: TP_FPGA93, TestPoint:TestPoint_Pad_D1.0mm, B.Cu at (168.1, 90.2)
- added TP3: TP_PPD5, TestPoint:TestPoint_Pad_D1.0mm, B.Cu at (193.1, 59.5)
- added TP30: TP_FPGA95, TestPoint:TestPoint_Pad_D1.0mm, B.Cu at (168.4, 95.2)
- added TP31: TP_FPGA97, TestPoint:TestPoint_Pad_D1.0mm, B.Cu at (166.9, 93.5)
- added TP32: TP_FPGA99, TestPoint:TestPoint_Pad_D1.0mm, B.Cu at (165.5, 95.2)
- added TP33: TP_FPGA101, TestPoint:TestPoint_Pad_D1.0mm, B.Cu at (165.7, 90.2)
- added TP34: TP_FPGA109, TestPoint:TestPoint_Pad_D1.0mm, B.Cu at (163.3, 90.2)
- added TP35: TP_FPGA111, TestPoint:TestPoint_Pad_D1.0mm, B.Cu at (163.4, 95.2)
- added TP36: TP_FPGA113, TestPoint:TestPoint_Pad_D1.0mm, B.Cu at (162.1, 93.5)
- added TP37: TP_FPGA115, TestPoint:TestPoint_Pad_D1.0mm, B.Cu at (160.8, 95.2)
- added TP38: TP_FPGA117, TestPoint:TestPoint_Pad_D1.0mm, B.Cu at (160.9, 90.2)
- added TP39: TP_FPGA155, TestPoint:TestPoint_Pad_D1.0mm, B.Cu at (149.5, 90.2)
- added TP4: TP_PPD4, TestPoint:TestPoint_Pad_D1.0mm, B.Cu at (191.8, 67.4)
- added TP40: TP_FPGA42, TestPoint:TestPoint_Pad_D1.0mm, B.Cu at (183.4, 98.4)
- added TP41: TP_FPGA44, TestPoint:TestPoint_Pad_D1.0mm, B.Cu at (183.6, 103.7)
- added TP42: TP_FPGA46, TestPoint:TestPoint_Pad_D1.0mm, B.Cu at (182.2, 102.0)
- added TP43: TP_FPGA48, TestPoint:TestPoint_Pad_D1.0mm, B.Cu at (180.8, 103.7)
- added TP44: TP_FPGA50, TestPoint:TestPoint_Pad_D1.0mm, B.Cu at (181.0, 98.4)
- added TP45: TP_FPGA52, TestPoint:TestPoint_Pad_D1.0mm, B.Cu at (179.4, 102.0)
- added TP46: TP_FPGA54, TestPoint:TestPoint_Pad_D1.0mm, B.Cu at (178.6, 98.4)
- added TP47: TP_FPGA122, TestPoint:TestPoint_Pad_D1.0mm, B.Cu at (159.4, 98.4)
- added TP48: TP_FPGA124, TestPoint:TestPoint_Pad_D1.0mm, B.Cu at (159.1, 103.7)
- added TP49: TP_FPGA128, TestPoint:TestPoint_Pad_D1.0mm, B.Cu at (157.6, 102.0)
- added TP5: TP_PPD3, TestPoint:TestPoint_Pad_D1.0mm, B.Cu at (190.5, 59.5)
- added TP50: TP_FPGA130, TestPoint:TestPoint_Pad_D1.0mm, B.Cu at (157.0, 98.4)
- added TP51: TP_FPGA132, TestPoint:TestPoint_Pad_D1.0mm, B.Cu at (156.1, 103.7)
- added TP52: TP_FPGA138, TestPoint:TestPoint_Pad_D1.0mm, B.Cu at (154.6, 102.0)
- added TP53: TP_FPGA142, TestPoint:TestPoint_Pad_D1.0mm, B.Cu at (153.4, 98.4)
- added TP54: TP_FPGA152, TestPoint:TestPoint_Pad_D1.0mm, B.Cu at (150.4, 98.4)
- added TP55: TP_FPGA156, TestPoint:TestPoint_Pad_D1.0mm, B.Cu at (149.2, 102.0)
- added TP6: TP_PPD2, TestPoint:TestPoint_Pad_D1.0mm, B.Cu at (189.2, 67.4)
- added TP7: TP_PPD1, TestPoint:TestPoint_Pad_D1.0mm, B.Cu at (188.0, 59.5)
- added TP8: TP_PPD0, TestPoint:TestPoint_Pad_D1.0mm, B.Cu at (186.8, 67.4)
- added TP9: TP_PACK, TestPoint:TestPoint_Pad_D1.0mm, B.Cu at (182.9, 59.5)
Connections:
- C54 pad 1: L_AUDIO -> Net-(SJ1-C)
- C56 pad 1: R_AUDIO -> Net-(SJ2-C)
- CN1 pad 11: unconnected-(CN1-AGREEN-Pad11) -> #AGREEN
- CN1 pad 15: unconnected-(CN1-ABLUE-Pad15) -> #ABLUE
- CN1 pad 16: unconnected-(CN1-/XCLKEN-Pad16) -> #XCLKEN
- CN1 pad 19: unconnected-(CN1-/C4-Pad19) -> #C4
- CN1 pad 28: unconnected-(CN1-BLANK-Pad28) -> #BLANK
- CN1 pad 33: unconnected-(CN1-/XCLK-Pad33) -> #XCLK
- CN1 pad 34: unconnected-(CN1-/C1-Pad34) -> #C1
- CN1 pad 7: unconnected-(CN1-ARED-Pad7) -> #ARED
- CN2 pad 13: unconnected-(CN2-SOG-Pad13) -> #SOG
- CN2 pad 14: unconnected-(CN2-TBASE-Pad14) -> #TBASE
- CN2 pad 16: unconnected-(CN2-PPOUT-Pad16) -> #PPOUT
- CN2 pad 17: unconnected-(CN2-/C3-Pad17) -> #C3
- CN2 pad 18: unconnected-(CN2-PBUSY-Pad18) -> #PBUSY
- CN2 pad 20: unconnected-(CN2-/PACK-Pad20) -> #PACK
- CN2 pad 23: unconnected-(CN2-PPD0-Pad23) -> #PPD0
- CN2 pad 24: unconnected-(CN2-PPD1-Pad24) -> #PPD1
- CN2 pad 25: unconnected-(CN2-PPD2-Pad25) -> #PPD2
- CN2 pad 26: unconnected-(CN2-PPD3-Pad26) -> #PPD3
- CN2 pad 27: unconnected-(CN2-PPD4-Pad27) -> #PPD4
- CN2 pad 28: unconnected-(CN2-PPD5-Pad28) -> #PPD5
- CN2 pad 29: unconnected-(CN2-PPD6-Pad29) -> #PPD6
- CN2 pad 30: unconnected-(CN2-PPD7-Pad30) -> #PPD7
- CN2 pad 31: unconnected-(CN2-/LED-Pad31) -> #LED
- CN2 pad 33: unconnected-(CN2-RAWLF-Pad33) -> RAWLF
- CN2 pad 35: unconnected-(CN2-RAWRT-Pad35) -> RAWRT
- U1 pad 101: unconnected-(U1-F19/PR17B-Pad101) -> #FPGA101
- U1 pad 109: unconnected-(U1-E19/PR14D-Pad109) -> #FPGA109
- U1 pad 111: unconnected-(U1-D20/PR14C-Pad111) -> #FPGA111
- U1 pad 113: unconnected-(U1-D19/PR14B-Pad113) -> #FPGA113
- U1 pad 115: unconnected-(U1-C20/PR14A-Pad115) -> #FPGA115
- U1 pad 117: unconnected-(U1-B20/PT67B-Pad117) -> #FPGA117
- U1 pad 122: unconnected-(U1-E6/PT6A-Pad122) -> #FPGA122
- U1 pad 124: unconnected-(U1-E5/PL11C-Pad124) -> #FPGA124
- U1 pad 128: unconnected-(U1-E4/PL8A-Pad128) -> #FPGA128
- U1 pad 130: unconnected-(U1-F1/PL26B-Pad130) -> #FPGA130
- U1 pad 132: unconnected-(U1-F3/PL23B-Pad132) -> #FPGA132
- U1 pad 138: unconnected-(U1-H4/PL20A-Pad138) -> #FPGA138
- U1 pad 142: unconnected-(U1-J4/PL29A-Pad142) -> #FPGA142
- U1 pad 152: unconnected-(U1-B3/PL5D-Pad152) -> #FPGA152
- U1 pad 155: unconnected-(U1-F2/PL23C-Pad155) -> #FPGA155
- U1 pad 156: unconnected-(U1-B2/PL14C-Pad156) -> #FPGA156
- U1 pad 41: unconnected-(U1-U16/PR47C-Pad41) -> #FPGA41
- U1 pad 42: unconnected-(U1-R1/PB4A-Pad42) -> #FPGA42
- U1 pad 44: unconnected-(U1-T1/PB4B-Pad44) -> #FPGA44
- U1 pad 46: unconnected-(U1-U1/PB6A-Pad46) -> #FPGA46
- U1 pad 48: unconnected-(U1-Y2/PB9B-Pad48) -> #FPGA48
- U1 pad 50: unconnected-(U1-W1/PB9A-Pad50) -> #FPGA50
- U1 pad 52: unconnected-(U1-V1/PB6B-Pad52) -> #FPGA52
- U1 pad 54: unconnected-(U1-M1/PL44B-Pad54) -> #FPGA54
- U1 pad 79: unconnected-(U1-M18/PR29D-Pad79) -> #FPGA79
- U1 pad 87: unconnected-(U1-K19/PR23B-Pad87) -> #FPGA87
- U1 pad 93: unconnected-(U1-H20/PR20B-Pad93) -> #FPGA93
- U1 pad 95: unconnected-(U1-G20/PR17D-Pad95) -> #FPGA95
- U1 pad 97: unconnected-(U1-G19/PR20A-Pad97) -> #FPGA97
- U1 pad 99: unconnected-(U1-F20/PR17C-Pad99) -> #FPGA99
- U4 pad 43: GND -> SPARE_IN5
- U4 pad 6: unconnected-(U4-1Y3-Pad6) -> SPARE_OUT3
Routing:
- net RAWLF: track 0.00 -> 127.7 mm
- net RAWRT: track 0.00 -> 124.7 mm, vias 0 -> 2
- net #ARED: track 0.00 -> 20.8 mm, vias 0 -> 2
- net #AGREEN: track 0.00 -> 15.0 mm, vias 0 -> 2
- net #XCLK: track 0.00 -> 15.0 mm, vias 0 -> 2
- net #SOG: track 0.00 -> 14.9 mm
- net #PPD4: track 0.00 -> 14.6 mm
- net #PPD2: track 0.00 -> 14.6 mm
- net #PPD6: track 0.00 -> 14.6 mm
- net #PPD0: track 0.00 -> 14.6 mm
- net #C3: track 0.00 -> 14.6 mm
- net #ABLUE: track 0.00 -> 14.4 mm, vias 0 -> 2
- net #C4: track 0.00 -> 14.4 mm, vias 0 -> 2
- net #LED: track 0.00 -> 14.4 mm
- net Net-(SJ2-C): track 0.00 -> 13.1 mm, vias 0 -> 1
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Other:
- board text added: "BeamBender BigBox Rev. 0.3"
- board text added: "FLT"
- board text added: "LEFT"
- board text added: "RAW"
- board text added: "Warning: Pin 41 is connected to a different IO on ColorLight i5 vs i9"
- board text removed: "BeamBender BigBox Rev. 0.2"

Commit message: Firmware 2026-10-30.03, BBLink 1.30, rev 0.3 production files and docs updates
Firmware (Firmware/: 2026-10-30.03 for the i9 and i5, standard and -c28, in place of 2026-10-28.04)
- Capture Clock on Display Info is steady: measured over 64 ms and shown to the nearest kHz, so it no longer flickers between two values.
- The input Frame Rate is timed against the card's own 27 MHz clock and holds steady (a PAL screen no longer flips between 49.91 and 49.92 Hz).
- The output frame rate is rounded like the input's: both read 50.38 Hz for a PAL screen on an NTSC-crystal machine with the -c28 firmware.
- Capture Width goes up to 800 and is shown in the screen's own pixels (up to 1360 on a Super-Hires screen); BB-800x600 on ECS shows all 800 columns.
- New defaults: Status Lines Hidden, Menu Position Bottom Right, Menu Background 50%.
- Settings record version 15 (since 2026-10-28.05): older records are not read, so back up with BBLink before updating from 2026-10-28.04 or earlier.
- The Amiga control link filters out short glitches on its lines.
- On-screen text in American spelling (Initializing, No RGB (gray), OSD Colors).

BBLink (BBLink/)
- bblink.lha: BBLink 1.30 (values in white on the live pages, as on the card), BBSurvey 1.12 (the 355-byte settings record), BBKeyCon, BBMode and BBProbe rebuilt for 2026-10-30.03. BBLag and BBScreen unchanged.
- README.md: the 2026-10-28.05 settings record, `[OSD Colors]` in backups (older `[OSD Colours]` files still load), values in white, examples for 1.30.
- Monitors/README.md: BB-800x600 on ECS shows all 800 columns. Monitors/bbmonitors.lha repacked; the drivers are unchanged.

Documentation
- Firmware/README.md: a new module's flash is unlocked through the card's JTAG header with `openFPGALoader -c ft232 --unprotect-flash` (one power cycle may be needed before the first write); the ecpdap and dev-board steps and the memory load (`-m`) are removed; sections reordered (adapter, software, unlock, write); the -c28 NTSC rate corrected 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
Parts:
- R49, R52: value 10K -> 8K2
- R51, R54: value 10K -> 20K
Changed lines of the file:
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@@
 			)
 		)
-		(property "Value" "10K"
+		(property "Value" "8K2"
 			(at 0 1.43 90)
 			(layer "F.Fab")
@@
 			)
 		)
-		(property "LCSC" "C25804"
+		(property "LCSC" "C25981"
 			(at 0 0 270)
 			(unlocked yes)
@@
 			)
 		)
-		(property "MPN" "0603WAF1002T5E"
+		(property "MPN" "0603WAF8201T5E"
 			(at 0 0 270)
 			(unlocked yes)
@@
 			)
 		)
-		(property "Value" "10K"
+		(property "Value" "20K"
 			(at 0 1.43 90)
 			(layer "F.Fab")
@@
 			)
 		)
-		(property "LCSC" "C25804"
+		(property "LCSC" "C4184"
 			(at 0 0 270)
 			(unlocked yes)
@@
 			)
 		)
-		(property "MPN" "0603WAF1002T5E"
+		(property "MPN" "0603WAF2002T5E"
 			(at 0 0 270)
 			(unlocked yes)
@@
 			)
 		)
-		(property "Value" "10K"
+		(property "Value" "20K"
 			(at 0 1.43 90)
 			(layer "F.Fab")
@@
 			)
 		)
-		(property "LCSC" "C25804"
+		(property "LCSC" "C4184"
 			(at 0 0 270)
 			(unlocked yes)
@@
 			)
 		)
-		(property "MPN" "0603WAF1002T5E"
+		(property "MPN" "0603WAF2002T5E"
 			(at 0 0 270)
 			(unlocked yes)
@@
 			)
 		)
-		(property "Value" "10K"
+		(property "Value" "8K2"
 			(at 0 1.43 90)
 			(layer "F.Fab")
@@
 			)
 		)
-		(property "LCSC" "C25804"
+		(property "LCSC" "C25981"
 			(at 0 0 270)
 			(unlocked yes)
@@
 			)
 		)
-		(property "MPN" "0603WAF1002T5E"
+		(property "MPN" "0603WAF8201T5E"
 			(at 0 0 270)
 			(unlocked yes)
@@
 			)
 		)
-		(attr smd)
+		(attr smd exclude_from_pos_files exclude_from_bom dnp)
 		(duplicate_pad_numbers_are_jumpers no)
 		(fp_line
